File: iqrfsim.brd (EAGLE design)
At the start: 37 x 19.5 mm, 6 parts

Commit message: Finish iqrfsim.brd for manufacture
Parts:
- removed G1: BATTERYTAP5-45, tagps:TAP5-45
- added GND, VIN: (no value), wirepad:1,6/0,9
- moved XC1 0.64 mm to (2.03, 13.3)
- moved U$1 0.13 mm to (33.0, 14.0)
- moved U$2 0.13 mm to (33.0, 5.08)
Connections:
- net GND: now also GND.1; no longer G1.-
- net VIN: now also VIN.1; no longer G1.+
Routing:
- net GND: track 18.2 -> 25.7 mm
- net IO/+3V: track 16.2 -> 15.4 mm
- net IO/ADC: track 20.1 -> 19.4 mm
- net IO/!SS: track 18.7 -> 18.1 mm
- net IO/SDO: track 29.7 -> 29.1 mm
- net IO/SDI: track 26.0 -> 25.3 mm
- net IO/CLK: track 23.0 -> 22.3 mm
Other:
- board size 37 x 19.5 mm -> 36.8 x 19.1 mm
Changed lines of the file:
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@@
 <setting verticaltext="up"/>
 </settings>
-<grid distance="10" unitdist="mil" unit="mil" style="lines" multiple="1" display="yes" altdistance="0.025" altunitdist="inch" altunit="inch"/>
+<grid distance="5" unitdist="mil" unit="mil" style="lines" multiple="1" display="yes" altdistance="0.025" altunitdist="inch" altunit="inch"/>
 <layers>
 <layer number="1" name="Top" color="4" fill="1" visible="yes" active="yes"/>
@@
 <board>
 <plain>
-<wire x1="0" y1="0" x2="37.008" y2="0" width="0" layer="20"/>
-<wire x1="37.008" y1="0" x2="37.008" y2="19.548" width="0" layer="20"/>
-<wire x1="37.008" y1="19.548" x2="0" y2="19.548" width="0" layer="20"/>
-<wire x1="0" y1="19.548" x2="0" y2="0" width="0" layer="20"/>
+<wire x1="0" y1="0" x2="36.83" y2="0" width="0" layer="20"/>
+<wire x1="36.83" y1="0" x2="36.83" y2="19.05" width="0" layer="20"/>
+<wire x1="36.83" y1="19.05" x2="0" y2="19.05" width="0" layer="20"/>
+<wire x1="0" y1="19.05" x2="0" y2="0" width="0" layer="20"/>
 <dimension x1="-1" y1="0" x2="-1" y2="20" x3="-9" y3="10" textsize="1.778" layer="1"/>
 <dimension x1="0" y1="-1" x2="40" y2="-1" x3="20" y3="-9" textsize="1.778" layer="1"/>
 <text x="17.272" y="1.27" size="0.8128" layer="51" font="vector">GND</text>
-<text x="20.066" y="0.508" size="0.8128" layer="51" font="vector">VIN</text>
+<text x="20.066" y="0.381" size="0.8128" layer="51" font="vector">VIN</text>
 <text x="21.59" y="1.27" size="0.8128" layer="51" font="vector">IO/+3V</text>
-<text x="24.686" y="0.442" size="0.8128" layer="51" font="vector">IO/ADC</text>
-<text x="17.018" y="18.034" size="0.8128" layer="51" font="vector">IO/!SS</text>
-<text x="19.304" y="17.018" size="0.8128" layer="51" font="vector">IO/CLK</text>
-<text x="21.844" y="18.034" size="0.8128" layer="51" font="vector">IO/SDI</text>
-<text x="24.638" y="17.018" size="0.8128" layer="51" font="vector">IO/SDO</text>
+<text x="24.638" y="0.381" size="0.8128" layer="51" font="vector">IO/ADC</text>
+<text x="17.018" y="17.78" size="0.8128" layer="51" font="vector">IO/!SS</text>
+<text x="19.304" y="16.637" size="0.8128" layer="51" font="vector">IO/CLK</text>
+<text x="21.844" y="17.78" size="0.8128" layer="51" font="vector">IO/SDI</text>
+<text x="24.638" y="16.637" size="0.8128" layer="51" font="vector">IO/SDO</text>
+<text x="27.432" y="12.7" size="0.8128" layer="51" font="vector">GND</text>
+<text x="27.559" y="5.08" size="0.8128" layer="51" font="vector">VIN</text>
 </plain>
 <attributes>
@@
 </autorouter>
 <elements>
-<element name="G1" library="tagps" package="TAP5-45" value="BATTERYTAP5-45" x="26.67" y="9.398" rot="R180"/>
 <element name="JP1" library="pinhead" package="1X04" value="" x="22.225" y="15.113"/>
 <element name="JP2" library="pinhead" package="1X04" value="" x="22.225" y="3.683" rot="R180"/>
-<element name="XC1" library="usbpiclib" package="SIM_8XPADS" value="SIM_8X" x="1.397" y="13.335"/>
-<element name="U$1" library="holes" package="2,8" value="" x="33.02" y="13.843"/>
-<element name="U$2" library="holes" package="2,8" value="" x="33.02" y="4.953"/>
+<element name="XC1" library="usbpiclib" package="SIM_8XPADS" value="SIM_8X" x="2.032" y="13.335"/>
+<element name="U$1" library="holes" package="2,8" value="" x="33.02" y="13.97"/>
+<element name="U$2" library="holes" package="2,8" value="" x="33.02" y="5.08"/>
+<element name="VIN" library="wirepad" package="1,6/0,9" value="" x="28.575" y="3.683"/>
+<element name="GND" library="wirepad" package="1,6/0,9" value="" x="28.575" y="15.113"/>
 </elements>
 <signals>
@@
 <contactref element="XC1" pad="8"/>
 <contactref element="JP1" pad="4"/>
-<wire x1="4.953" y1="5.715" x2="1.397" y2="5.715" width="0.4064" layer="1"/>
+<wire x1="4.953" y1="5.715" x2="2.032" y2="5.715" width="0.4064" layer="1"/>
 <wire x1="26.035" y1="15.113" x2="26.035" y2="13.081" width="0.4064" layer="16"/>
-<wire x1="26.035" y1="13.081" x2="25.4" y2="12.446" width="0.4064" layer="16"/>
-<wire x1="25.4" y1="12.446" x2="24.003" y2="12.446" width="0.4064" layer="16"/>
-<wire x1="24.003" y1="12.446" x2="20.574" y2="9.017" width="0.4064" layer="16"/>
-<wire x1="20.574" y1="9.017" x2="9.525" y2="9.017" width="0.4064" layer="16"/>
-<wire x1="9.525" y1="9.017" x2="6.223" y2="5.715" width="0.4064" layer="16"/>
 <via x="4.953" y="5.715" extent="1-16" drill="0.6"/>
-<wire x1="4.953" y1="5.715" x2="6.223" y2="5.715" width="0.4064" layer="16"/>
+<wire x1="4.953" y1="5.715" x2="6.477" y2="5.715" width="0.4064" layer="16"/>
+<wire x1="26.035" y1="13.081" x2="21.463" y2="8.509" width="0.4064" layer="16"/>
+<wire x1="21.463" y1="8.509" x2="9.271" y2="8.509" width="0.4064" layer="16"/>
+<wire x1="9.271" y1="8.509" x2="6.477" y2="5.715" width="0.4064" layer="16"/>
 </signal>
 <signal name="IO/CLK">
 <contactref element="XC1" pad="6"/>
 <contactref element="JP1" pad="2"/>
-<wire x1="4.953" y1="10.795" x2="1.397" y2="10.795" width="0.4064" layer="1"/>
+<wire x1="4.953" y1="10.795" x2="2.032" y2="10.795" width="0.4064" layer="1"/>
 <wire x1="20.955" y1="12.319" x2="20.955" y2="15.113" width="0.4064" layer="16"/>
 <via x="4.953" y="10.795" extent="1-16" drill="0.6"/>
@@
 <contactref element="XC1" pad="7"/>
 <contactref element="JP1" pad="3"/>
-<wire x1="4.953" y1="8.255" x2="1.397" y2="8.255" width="0.4064" layer="1"/>
+<wire x1="4.953" y1="8.255" x2="2.032" y2="8.255" width="0.4064" layer="1"/>
 <wire x1="23.495" y1="13.335" x2="19.939" y2="9.779" width="0.4064" layer="16"/>
 <wire x1="23.495" y1="13.335" x2="23.495" y2="15.113" width="0.4064" layer="16"/>
@@
 <contactref element="XC1" pad="5"/>
 <contactref element="JP1" pad="1"/>
-<wire x1="4.953" y1="13.335" x2="1.397" y2="13.335" width="0.4064" layer="1"/>
+<wire x1="4.953" y1="13.335" x2="2.032" y2="13.335" width="0.4064" layer="1"/>
 <wire x1="18.415" y1="13.462" x2="18.415" y2="15.113" width="0.4064" layer="16"/>
 <via x="4.953" y="13.335" extent="1-16" drill="0.6"/>
@@
 <contactref element="XC1" pad="2"/>
 <contactref element="JP2" pad="2"/>
-<wire x1="23.495" y1="3.683" x2="23.495" y2="5.461" width="0.4064" layer="1"/>
-<wire x1="23.495" y1="5.461" x2="18.161" y2="10.795" width="0.4064" layer="1"/>
-<wire x1="18.161" y1="10.795" x2="11.2394" y2="10.795" width="0.4064" layer="1"/>
+<wire x1="17.78" y1="10.795" x2="11.8744" y2="10.795" width="0.4064" layer="1"/>
+<wire x1="17.78" y1="10.795" x2="23.495" y2="5.08" width="0.4064" layer="1"/>
+<wire x1="23.495" y1="5.08" x2="23.495" y2="3.683" width="0.4064" layer="1"/>
 </signal>
 <signal name="IO/ADC">
 <contactref element="XC1" pad="1"/>
 <contactref element="JP2" pad="1"/>
-<wire x1="16.637" y1="13.335" x2="11.2394" y2="13.335" width="0.4064" layer="1"/>
+<wire x1="16.637" y1="13.335" x2="11.8744" y2="13.335" width="0.4064" layer="1"/>
 <wire x1="26.035" y1="3.683" x2="26.035" y2="5.842" width="0.4064" layer="1"/>
 <wire x1="26.035" y1="5.842" x2="25.146" y2="6.731" width="0.4064" layer="1"/>
@@
 <contactref element="XC1" pad="3"/>
 <contactref element="JP2" pad="3"/>
-<contactref element="G1" pad="+"/>
 <wire x1="20.955" y1="3.683" x2="20.955" y2="6.35" width="0.4064" layer="1"/>
 <wire x1="20.955" y1="6.35" x2="19.05" y2="8.255" width="0.4064" layer="1"/>
-<wire x1="19.05" y1="8.255" x2="11.2394" y2="8.255" width="0.4064" layer="1"/>
-<wire x1="29.21" y1="9.398" x2="27.305" y2="7.493" width="0.4064" layer="16"/>
-<wire x1="27.305" y1="7.493" x2="21.336" y2="7.493" width="0.4064" layer="16"/>
-<wire x1="21.336" y1="7.493" x2="20.955" y2="7.112" width="0.4064" layer="16"/>
-<wire x1="20.955" y1="7.112" x2="20.955" y2="3.683" width="0.4064" layer="16"/>
+<wire x1="19.05" y1="8.255" x2="11.8744" y2="8.255" width="0.4064" layer="1"/>
+<wire x1="20.955" y1="5.842" x2="20.955" y2="3.683" width="0.4064" layer="16"/>
+<contactref element="VIN" pad="1"/>
+<wire x1="28.575" y1="3.683" x2="28.575" y2="6.223" width="0.4064" layer="16"/>
+<wire x1="20.955" y1="5.842" x2="21.717" y2="6.604" width="0.4064" layer="16"/>
+<wire x1="21.717" y1="6.604" x2="28.194" y2="6.604" width="0.4064" layer="16"/>
+<wire x1="28.194" y1="6.604" x2="28.575" y2="6.223" width="0.4064" layer="16"/>
 </signal>
 <signal name="GND">
 <contactref element="XC1" pad="4"/>
 <contactref element="JP2" pad="4"/>
-<contactref element="G1" pad="-"/>
 <wire x1="18.415" y1="3.683" x2="18.415" y2="5.588" width="0.4064" layer="1"/>
 <wire x1="18.415" y1="5.588" x2="18.288" y2="5.715" width="0.4064" layer="1"/>
-<wire x1="18.288" y1="5.715" x2="11.2394" y2="5.715" width="0.4064" layer="1"/>
-<wire x1="22.86" y1="9.398" x2="21.717" y2="8.255" width="0.4064" layer="16"/>
-<wire x1="21.717" y1="8.255" x2="19.177" y2="8.255" width="0.4064" layer="16"/>
-<wire x1="19.177" y1="8.255" x2="18.415" y2="7.493" width="0.4064" layer="16"/>
-<wire x1="18.415" y1="7.493" x2="18.415" y2="3.683" width="0.4064" layer="16"/>
+<wire x1="18.288" y1="5.715" x2="11.8744" y2="5.715" width="0.4064" layer="1"/>
+<contactref element="GND" pad="1"/>
+<wire x1="28.575" y1="15.113" x2="28.575" y2="13.97" width="0.4064" layer="16"/>
+<wire x1="28.575" y1="13.97" x2="22.098" y2="7.493" width="0.4064" layer="16"/>
+<wire x1="22.098" y1="7.493" x2="19.431" y2="7.493" width="0.4064" layer="16"/>
+<wire x1="19.431" y1="7.493" x2="18.415" y2="6.477" width="0.4064" layer="16"/>
+<wire x1="18.415" y1="6.477" x2="18.415" y2="3.683" width="0.4064" layer="16"/>
 </signal>
 </signals>
